Commit message: Add transition logic for gesture scripts and safety bridge waypoints

File: pepper_ign_moveit2/pepper_robot_description/urdf/pepper_robot.urdf (robot description, URDF)
Before this commit: robot pepper_robot, 83 links, 82 joints
Links:
- link LFinger11_link: mass 5e-3 -> 0.05
- link LFinger12_link: mass 5e-3 -> 0.05
- link LFinger13_link: mass 5e-3 -> 0.05
- link LFinger21_link: mass 5e-3 -> 0.05
- link LFinger22_link: mass 5e-3 -> 0.05
- link LFinger23_link: mass 5e-3 -> 0.05
- link LFinger31_link: mass 5e-3 -> 0.05
- link LFinger32_link: mass 5e-3 -> 0.05
- link LFinger33_link: mass 5e-3 -> 0.05
- link LFinger41_link: mass 5e-3 -> 0.05
- link LFinger42_link: mass 5e-3 -> 0.05
- link LFinger43_link: mass 5e-3 -> 0.05
- link LThumb1_link: mass 5e-3 -> 0.05
- link LThumb2_link: mass 5e-3 -> 0.05
- link RFinger11_link: mass 5e-3 -> 0.05
- link RFinger12_link: mass 5e-3 -> 0.05
- link RFinger13_link: mass 5e-3 -> 0.05
- link RFinger21_link: mass 5e-3 -> 0.05
- link RFinger22_link: mass 5e-3 -> 0.05
- link RFinger23_link: mass 5e-3 -> 0.05
- link RFinger31_link: mass 5e-3 -> 0.05
- link RFinger32_link: mass 5e-3 -> 0.05
- link RFinger33_link: mass 5e-3 -> 0.05
- link RFinger41_link: mass 5e-3 -> 0.05
- link RFinger42_link: mass 5e-3 -> 0.05
- link RFinger43_link: mass 5e-3 -> 0.05
- link RThumb1_link: mass 5e-3 -> 0.05
- link RThumb2_link: mass 5e-3 -> 0.05
- link l_gripper: mass 1e-5 -> 0.05
- link r_gripper: mass 1e-5 -> 0.05
Joints:
- joint LHand: limit lower=0.02 upper=0.98 effort=0.144 velocity=12.56 -> lower=0.02 upper=0.98 effort=5.428 velocity=12.56

Commit message: allowed some modular functionality into gesture_manager+looping eventually

File: pepper_ign_moveit2/pepper_robot_description/urdf/pepper_robot.urdf (robot description, URDF)
Before this commit: robot pepper_robot, 83 links, 82 joints
Links:
- link LFinger11_link: mass 0.05 -> 5e-3
- link LFinger12_link: mass 0.05 -> 5e-3
- link LFinger13_link: mass 0.05 -> 5e-3
- link LFinger21_link: mass 0.05 -> 5e-3
- link LFinger22_link: mass 0.05 -> 5e-3
- link LFinger23_link: mass 0.05 -> 5e-3
- link LFinger31_link: mass 0.05 -> 5e-3
- link LFinger32_link: mass 0.05 -> 5e-3
- link LFinger33_link: mass 0.05 -> 5e-3
- link LFinger41_link: mass 0.05 -> 5e-3
- link LFinger42_link: mass 0.05 -> 5e-3
- link LFinger43_link: mass 0.05 -> 5e-3
- link LThumb1_link: mass 0.05 -> 5e-3
- link LThumb2_link: mass 0.05 -> 5e-3
- link RFinger11_link: mass 0.05 -> 5e-3
- link RFinger12_link: mass 0.05 -> 5e-3
- link RFinger13_link: mass 0.05 -> 5e-3
- link RFinger21_link: mass 0.05 -> 5e-3
- link RFinger22_link: mass 0.05 -> 5e-3
- link RFinger23_link: mass 0.05 -> 5e-3
- link RFinger31_link: mass 0.05 -> 5e-3
- link RFinger32_link: mass 0.05 -> 5e-3
- link RFinger33_link: mass 0.05 -> 5e-3
- link RFinger41_link: mass 0.05 -> 5e-3
- link RFinger42_link: mass 0.05 -> 5e-3
- link RFinger43_link: mass 0.05 -> 5e-3
- link RThumb1_link: mass 0.05 -> 5e-3
- link RThumb2_link: mass 0.05 -> 5e-3
- link l_gripper: mass 0.05 -> 1e-5
- link r_gripper: mass 0.05 -> 1e-5
Joints:
- joint LHand: limit lower=0.02 upper=0.98 effort=5.428 velocity=12.56 -> lower=0.02 upper=0.98 effort=0.144 velocity=12.56
